Commit message: Add interactive URDF 3D viewer

File: franky_amr.urdf (robot description, URDF)
Before this commit: robot franky_amr, 7 links, 6 joints
Links:
- added link base_footprint
- link base_link: mass None -> 0.82573504; geometry collision box size=0.18 0.14 0.08; visual mesh filename=meshes/base_link.STL
- link caster_front_link: mass None -> 1.44379265037903E-06; geometry collision sphere radius=0.005; visual mesh filename=meshes/caster_front_link.STL
- link caster_rear_link: mass None -> 1.44379265037902E-06; geometry collision sphere radius=0.005; visual mesh filename=meshes/caster_rear_link.STL
- link imu_link: mass None -> 0.000528415362211671
- link wheel_left_link: mass None -> 0.0530086043217644; geometry collision sphere radius=0.033; visual mesh filename=meshes/wheel_left_link.STL
- link wheel_right_link: mass None -> 0.0530086090966721; geometry collision sphere radius=0.033; visual mesh filename=meshes/wheel_right_link.STL
Joints:
- added joint base_joint: type fixed, parent base_footprint, child base_link, origin xyz=0 0 0.033 rpy=0 0 0
- joint caster_front_joint: origin xyz=0.10 0 -0.015 rpy=0 0 0 -> xyz=0.04755 0 -0.0275 rpy=0 0 0
- joint caster_rear_joint: origin xyz=-0.10 0 -0.015 rpy=0 0 0 -> xyz=-0.04755 0 -0.0275 rpy=0 0 0
- joint imu_joint: origin xyz=0 0 0.05 rpy=0 0 0 -> xyz=0 0 0.0698986241758014 rpy=0 0 0
- joint wheel_left_joint: origin xyz=0 0.085 0 rpy=0 0 0 -> xyz=0 0.07 0.0 rpy=0 0 0
- joint wheel_right_joint: origin xyz=0 -0.085 0 rpy=0 0 0 -> xyz=0 -0.07 0.0 rpy=0 0 0
